Commit message: Fixed Gazebo issue intertial added to links and model now spawns correctly in Gazebo

File: simulation_ws/src/cart_sim/urdf/cart_model.urdf (robot description, URDF)
Before this commit: robot cart_model, 4 links, 3 joints
Links:
- added link world
- link D455_link: mass 10 -> None
- link base_link: mass 10 -> None
- link lms_link: mass 10 -> None
- link tim_link: mass 10 -> None
Joints:
- added joint world_to_base: type fixed, parent world, child base_link, origin xyz=0 0 0
